File: measure water tank.kicad_sch (KiCad schematic)
At the start: 14 parts, among them J1 Jack-DC, J2 Conn_ARM_SWD_TagConnect_TC2030, U1 SPX3819M5-L, U2 SPX3819M5-L, U3 ESP32-S3-MINI-1U

Commit message: add: ch340 changed: esp32
Parts:
- removed F2: 600mA, symbol Device:Fuse
- removed J2: Conn_ARM_SWD_TagConnect_TC2030, Connector:Tag-Connect_TC2030-IDC-FP_2x03_P1.27mm_Vertical, symbol Connector:Conn_ARM_SWD_TagConnect_TC2030
- added C7: 0.1nF/25v, Capacitor_SMD:C_1206_3216Metric, symbol Device:C
- C1, C2, C3: footprint (none) -> Capacitor_SMD:C_1206_3216Metric
- C4: value 1uf -> 10nF/6.3V; footprint (none) -> Capacitor_SMD:C_1206_3216Metric
- C5: value 10nF -> 470pf; footprint (none) -> Capacitor_SMD:C_1206_3216Metric
- F1: footprint (none) -> Fuse:Fuse_Bourns_MF-RG300
- J1: footprint (none) -> Connector_BarrelJack:BarrelJack_Horizontal
- R1, R2: footprint (none) -> Resistor_SMD:R_1206_3216Metric
Connections:
- net +12V: now also C3.1, U1.1 (IN), U1.3 (EN)
- net +3v3: now also C7.1
- net GND: now also C3.2, C7.2
- net usb_5v: now reaches C2.1, F1.2
- net ch340c-rx: now reaches U3.39 (TXD0)
- net ch340c-tx: now reaches U3.40 (RXD0)
Other:
- added sheet usb (power and esp12.kicad_sch)

Commit message: add: protector de estatica
Parts:
- added C6: 0.1nF/25v, Capacitor_SMD:C_1206_3216Metric, symbol Device:C
- added R6: 0, symbol Device:R_US
- added SW1: SW_Push, symbol Switch:SW_Push
Connections:
- net GND: now also C6.1, SW1.1
- net Gpio0: now reaches U3.4 (IO0)
- net EN: now reaches U3.45 (EN)
- net EN: now also R6.2
- net usb_5v: no longer names the net of C2.1, F1.2
- new net: C6.2, R6.1, SW1.2

Commit message: del: elimine el ch340 y conecte el usb directamente
Parts:
- added D2: yellow, LED_SMD:LED_0603_1608Metric, symbol SparkFun-LED:LED_Red_0603
- added D3: Red, LED_SMD:LED_0603_1608Metric, symbol SparkFun-LED:LED_Red_0603
- added D4: blue, LED_SMD:LED_0603_1608Metric, symbol SparkFun-LED:LED_Red_0603
- added JP1: ~, Jumper:SolderJumper-2_P1.3mm_Bridged_Pad1.0x1.5mm, symbol SparkFun-Jumper:SolderJumper_2_Bridged
- added R11, R4, R8: 4.7k, Resistor_SMD:R_0402_1005Metric, symbol SparkFun-Resistor:4.7k_0402
- added R3: 10k, Resistor_SMD:R_0402_1005Metric, symbol Device:R_US
- C1, C2, C3, C4, C5, C6, C7: footprint Capacitor_SMD:C_1206_3216Metric -> Capacitor_SMD:C_0402_1005Metric
- R1, R2: footprint Resistor_SMD:R_1206_3216Metric -> Resistor_SMD:R_0402_1005Metric
- R6: footprint (none) -> Resistor_SMD:R_0402_1005Metric
- SW1: footprint (none) -> Button_Switch_THT:SW_PUSH_6mm
Connections:
- net +12V: now also R4.1; no longer C3.1, U1.1 (IN), U1.3 (EN)
- net +3v3: now also JP1.2 (B), R3.1
- net +5v: now also C3.1, U1.1 (IN), U1.3 (EN), D2.1 (K), D3.1 (K); no longer C1.1, R1.1, U2.5 (OUT)
- net EN: now also R3.2
- net GND: now also D4.1 (K)
- net at C2.2, U2.1 (IN): no longer U2.3 (EN)
- net ESP8/SDA: now reaches U3.12 (IO8)
- net ESP9/SCL: now reaches U3.13 (IO9)
- net d-: now reaches U3.23 (IO19)
- net d+: now reaches U3.24 (IO20)
- net ch340c-rx: no longer names the net of U3.39 (TXD0)
- net ch340c-tx: no longer names the net of U3.40 (RXD0)
- new net: D4.2 (A), R11.2
- new net: C1.1, R1.1, R8.2, U2.5 (OUT)
- new net: D3.2 (A), R4.2
- new net: D2.2 (A), R8.1
- new net: JP1.1 (A), R11.1
- new net led_control: U2.3 (EN)
Other:
- moved on the sheet: C6, C7, R6, SW1, U3
